File: hardware/ATTiny85 5LED R1.sch (EAGLE design)
At the start: 9 parts, among them U1 TINY85-20-DIP

Commit message: updating eagle files
Parts:
- S2: value MOMENTARY-SWITCH-SPST-PTH-6.0MM -> (none); device SparkFun-Switches:MOMENTARY-SWITCH-SPST-PTH-6.0MM -> adafruit:SWITCH_PUSHBUTTONEVQ-PE
Connections:
- net GND: now also S2.P$1; no longer S2.2
- net PB5: now also S2.P$2; no longer S2.1
Changed lines of the file:
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@@
 <?xml version="1.0" encoding="utf-8"?>
 <!DOCTYPE eagle SYSTEM "eagle.dtd">
-<eagle version="8.3.2">
+<eagle version="9.4.1">
 <drawing>
 <settings>
@@
 <part name="BT1" library="SparkFun-Batteries" deviceset="BATTERY" device="-20MM_PTH"/>
 <part name="S1" library="SparkFun-Switches" deviceset="SWITCH-SPDT" device="-PTH-11.6X4.0MM-KIT"/>
-<part name="S2" library="SparkFun-Switches" deviceset="MOMENTARY-SWITCH-SPST" device="-PTH-6.0MM" value=""/>
+<part name="S2" library="adafruit" deviceset="SWITCH_PUSHBUTTON" device="EVQ-PE"/>
 <part name="GND2" library="SparkFun-PowerSymbols" deviceset="GND" device=""/>
 <part name="GND3" library="SparkFun-PowerSymbols" deviceset="GND" device=""/>
@@
 </plain>
 <instances>
-<instance part="FRAME1" gate="G$1" x="0" y="0"/>
-<instance part="GND1" gate="1" x="111.76" y="83.82"/>
-<instance part="U1" gate="G$1" x="132.08" y="96.52"/>
-<instance part="D3" gate="G$1" x="226.06" y="147.32" rot="R90"/>
-<instance part="D4" gate="G$1" x="226.06" y="129.54" rot="R90"/>
-<instance part="D5" gate="G$1" x="226.06" y="111.76" rot="R90"/>
-<instance part="D6" gate="G$1" x="226.06" y="93.98" rot="R90"/>
-<instance part="D7" gate="G$1" x="226.06" y="76.2" rot="R90"/>
-<instance part="GND4" gate="1" x="236.22" y="139.7" rot="MR0"/>
-<instance part="GND5" gate="1" x="236.22" y="121.92" rot="MR0"/>
-<instance part="GND6" gate="1" x="236.22" y="104.14" rot="MR0"/>
-<instance part="GND7" gate="1" x="236.22" y="86.36" rot="MR0"/>
-<instance part="GND8" gate="1" x="236.22" y="68.58" rot="MR0"/>
-<instance part="SUPPLY2" gate="G$1" x="111.76" y="109.22"/>
-<instance part="BT1" gate="G$1" x="30.48" y="132.08" rot="R180"/>
-<instance part="S1" gate="1" x="43.18" y="132.08"/>
-<instance part="S2" gate="G$1" x="35.56" y="45.72"/>
-<instance part="GND2" gate="1" x="45.72" y="38.1"/>
-<instance part="GND3" gate="1" x="20.32" y="124.46"/>
-<instance part="SUPPLY1" gate="G$1" x="53.34" y="127" rot="R180"/>
+<instance part="FRAME1" gate="G$1" x="0" y="0" smashed="yes">
+<attribute name="DRAWING_NAME" x="181.61" y="11.43" size="2.54" layer="94" font="vector"/>
+<attribute name="LAST_DATE_TIME" x="181.61" y="6.35" size="2.286" layer="94" font="vector"/>
+<attribute name="SHEET" x="195.58" y="1.27" size="2.54" layer="94" font="vector"/>
+<attribute name="CNAME" x="181.61" y="16.51" size="2.54" layer="94" font="vector"/>
+<attribute name="DESIGNER" x="226.26" y="6.35" size="2.54" layer="94" font="vector"/>
+<attribute name="CREVISION" x="234.92" y="1.17" size="2.54" layer="94" font="vector"/>
+</instance>
+<instance part="GND1" gate="1" x="111.76" y="83.82" smashed="yes">
+<attribute name="VALUE" x="111.76" y="83.566" size="1.778" layer="96" align="top-center"/>
+</instance>
+<instance part="U1" gate="G$1" x="132.08" y="96.52" smashed="yes">
+<attribute name="VALUE" x="119.38" y="86.36" size="1.778" layer="96"/>
+<attribute name="NAME" x="119.38" y="106.68" size="1.778" layer="95"/>
+</instance>
+<instance part="D3" gate="G$1" x="226.06" y="147.32" smashed="yes" rot="R90">
+<attribute name="NAME" x="230.632" y="143.891" size="1.778" layer="95" font="vector" rot="R180"/>
+<attribute name="VALUE" x="230.632" y="149.225" size="1.778" layer="96" font="vector" rot="R180" align="top-left"/>
+</instance>
+<instance part="D4" gate="G$1" x="226.06" y="129.54" smashed="yes" rot="R90">
+<attribute name="NAME" x="230.632" y="126.111" size="1.778" layer="95" font="vector" rot="R180"/>
+<attribute name="VALUE" x="230.632" y="131.445" size="1.778" layer="96" font="vector" rot="R180" align="top-left"/>
+</instance>
+<instance part="D5" gate="G$1" x="226.06" y="111.76" smashed="yes" rot="R90">
+<attribute name="NAME" x="230.632" y="108.331" size="1.778" layer="95" font="vector" rot="R180"/>
+<attribute name="VALUE" x="230.632" y="113.665" size="1.778" layer="96" font="vector" rot="R180" align="top-left"/>
+</instance>
+<instance part="D6" gate="G$1" x="226.06" y="93.98" smashed="yes" rot="R90">
+<attribute name="NAME" x="230.632" y="90.551" size="1.778" layer="95" font="vector" rot="R180"/>
+<attribute name="VALUE" x="230.632" y="95.885" size="1.778" layer="96" font="vector" rot="R180" align="top-left"/>
+</instance>
+<instance part="D7" gate="G$1" x="226.06" y="76.2" smashed="yes" rot="R90">
+<attribute name="NAME" x="230.632" y="72.771" size="1.778" layer="95" font="vector" rot="R180"/>
+<attribute name="VALUE" x="230.632" y="78.105" size="1.778" layer="96" font="vector" rot="R180" align="top-left"/>
+</instance>
+<instance part="GND4" gate="1" x="236.22" y="139.7" smashed="yes" rot="MR0">
+<attribute name="VALUE" x="236.22" y="139.446" size="1.778" layer="96" rot="MR0" align="top-center"/>
+</instance>
+<instance part="GND5" gate="1" x="236.22" y="121.92" smashed="yes" rot="MR0">
+<attribute name="VALUE" x="236.22" y="121.666" size="1.778" layer="96" rot="MR0" align="top-center"/>
+</instance>
+<instance part="GND6" gate="1" x="236.22" y="104.14" smashed="yes" rot="MR0">
+<attribute name="VALUE" x="236.22" y="103.886" size="1.778" layer="96" rot="MR0" align="top-center"/>
+</instance>
+<instance part="GND7" gate="1" x="236.22" y="86.36" smashed="yes" rot="MR0">
+<attribute name="VALUE" x="236.22" y="86.106" size="1.778" layer="96" rot="MR0" align="top-center"/>
+</instance>
+<instance part="GND8" gate="1" x="236.22" y="68.58" smashed="yes" rot="MR0">
+<attribute name="VALUE" x="236.22" y="68.326" size="1.778" layer="96" rot="MR0" align="top-center"/>
+</instance>
+<instance part="SUPPLY2" gate="G$1" x="111.76" y="109.22" smashed="yes">
+<attribute name="VALUE" x="111.76" y="112.014" size="1.778" layer="96" align="bottom-center"/>
+</instance>
+<instance part="BT1" gate="G$1" x="30.48" y="132.08" smashed="yes" rot="R180">
+<attribute name="NAME" x="30.48" y="127.762" size="1.778" layer="95" font="vector" rot="R180" align="bottom-center"/>
+<attribute name="VALUE" x="30.48" y="136.398" size="1.778" layer="96" font="vector" rot="R180" align="top-center"/>
+</instance>
+<instance part="S1" gate="1" x="43.18" y="132.08" smashed="yes">
+<attribute name="NAME" x="44.45" y="135.128" size="1.778" layer="95" font="vector" align="bottom-center"/>
+<attribute name="VALUE" x="44.196" y="128.778" size="1.778" layer="96" font="vector" align="top-center"/>
+</instance>
+<instance part="S2" gate="G$1" x="35.56" y="45.72" smashed="yes">
+<attribute name="NAME" x="35.56" y="47.244" size="1.778" layer="95" font="vector" align="bottom-center"/>
+<attribute name="VALUE" x="35.56" y="45.212" size="1.778" layer="96" font="vector" align="top-center"/>
+</instance>
+<instance part="GND2" gate="1" x="25.4" y="38.1" smashed="yes">
+<attribute name="VALUE" x="25.4" y="37.846" size="1.778" layer="96" align="top-center"/>
+</instance>
+<instance part="GND3" gate="1" x="20.32" y="124.46" smashed="yes">
+<attribute name="VALUE" x="20.32" y="124.206" size="1.778" layer="96" align="top-center"/>
+</instance>
+<instance part="SUPPLY1" gate="G$1" x="53.34" y="127" smashed="yes" rot="R180">
+<attribute name="VALUE" x="53.34" y="124.206" size="1.778" layer="96" rot="R180" align="bottom-center"/>
+</instance>
 </instances>
 <busses>
@@
 </segment>
 <segment>
-<pinref part="S2" gate="G$1" pin="2"/>
-<pinref part="GND2" gate="1" pin="GND"/>
-<wire x1="40.64" y1="45.72" x2="45.72" y2="45.72" width="0.1524" layer="91"/>
-<wire x1="45.72" y1="45.72" x2="45.72" y2="40.64" width="0.1524" layer="91"/>
-</segment>
-<segment>
 <pinref part="BT1" gate="G$1" pin="-"/>
 <pinref part="GND3" gate="1" pin="GND"/>
@@
 <wire x1="20.32" y1="132.08" x2="20.32" y2="127" width="0.1524" layer="91"/>
 </segment>
+<segment>
+<pinref part="GND2" gate="1" pin="GND"/>
+<wire x1="25.4" y1="40.64" x2="25.4" y2="45.72" width="0.1524" layer="91"/>
+<pinref part="S2" gate="G$1" pin="P$1"/>
+<wire x1="25.4" y1="45.72" x2="30.48" y2="45.72" width="0.1524" layer="91"/>
+</segment>
 </net>
 <net name="VCC" class="0">
@@
 <segment>
 <pinref part="S1" gate="1" pin="S"/>
+<wire x1="48.26" y1="129.54" x2="53.34" y2="129.54" width="0.1524" layer="91"/>
 <pinref part="SUPPLY1" gate="G$1" pin="VCC"/>
-<wire x1="48.26" y1="129.54" x2="53.34" y2="129.54" width="0.1524" layer="91"/>
 <wire x1="53.34" y1="129.54" x2="53.34" y2="127" width="0.1524" layer="91"/>
 </segment>
@@
 </segment>
 <segment>
-<pinref part="S2" gate="G$1" pin="1"/>
-<wire x1="30.48" y1="45.72" x2="25.4" y2="45.72" width="0.1524" layer="91"/>
-<label x="25.4" y="45.72" size="1.27" layer="95" rot="MR0" xref="yes"/>
-</segment>
-</net>
+<pinref part="S2" gate="G$1" pin="P$2"/>
+<wire x1="40.64" y1="45.72" x2="45.72" y2="45.72" width="0.1524" layer="91"/>
+<label x="45.72" y="45.72" size="1.27" layer="95" xref="yes"/>
+</segment>
+</net>
